File: 1inch-photodetector.kicad_pcb (KiCad board)
At the start: 4 copper layers, 25.4 x 25.4 mm, 23 parts, among them J1 Conn_01x03, J2 Conn_Coaxial, U1 ADA4898-2, U2 LT3032IDE-12

Commit message: Add 'Do not touch artwork' disclaimer (#15)
- Added more disclaimers for assembly
Other:
- board text added: "Manufacturing Instruction: - Material FR-4 - Finished thickness: 1.57 mm ± 0.13 mm - PCBs must be RoHS compliant - Do not edit artwork, e.g. to add logos or order numbers - Clean to meet IPC J-STD-001E, Class 2 after assembly"
Changed lines of the file:
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@@
+		)
+	)
+	(gr_text "Manufacturing Instruction:\n- Material FR-4\n- Finished thickness: 1.57 mm ± 0.13 mm\n- PCBs must be RoHS compliant\n- Do not edit artwork, e.g. to add logos\n   or order numbers\n- Clean to meet IPC J-STD-001E, Class 2\n   after assembly"
+		(at 150 45 0)
+		(layer "Cmts.User")
+		(effects
+			(font
+				(size 1 1)
+				(thickness 0.15)
+			)
+			(justify left bottom)
 		)
 	)
