File: 1inch-photodetector.kicad_pcb (KiCad board)
At the start: 4 copper layers, 25.4 x 25.4 mm, 23 parts, among them J1 Conn_01x03, J2 Conn_Coaxial, U1 ADA4898-2, U2 LT3032IDE-12

Commit message: Update components
Routing:
- net /V-: track 8.77 -> 6.72 mm
